File: bitaxeHex.kicad_pcb (KiCad board)
At the start: 4 copper layers, 84.5 x 129.5 mm, 360 parts, among them J1 Conn_01x01, J2 Conn_01x01, J3 Conn_02x05_Odd_Even, J4 TC2030-IDC, J5 Conn_01x04, J6 Conn_01x06, J7 USB_C_Receptacle_USB2.0, J8 Conn_01x04, J9 Conn_01x04, SW1 SWITCH-SPST, SW2 SWITCH-SPST, U1 LMR54410, U10 AP7331, U11 AP7331, U12 BM1366_mode1, U13 BM1366_mode1, U14 25MHz, U15 TLV3544, U16 AP7331, U17 AP7331, U18 BM1366_mode0, U19 25MHz, U2 RT9080-33GJ5, U20 BM1366_mode0, U21 TLV3544, U22 BM1366_mode1, U23 AP7331, U24 AP7331, U25 BM1366_mode1, U26 25MHz, U3 TPS546D24ARVFR, U4 MIC5504, U5 SN74AVC4T774, U6 ESP32-S3-WROOM-1, U7 TMP1075, U8 TMP1075, U9 EMC2302, Y1 32.768kHz

Commit message: Add special version for OSMU
Parts:
- added REF**: OSMU_logo_mask, bitaxe:OSMU_logo_mask, F.Cu at (55.5, 132.8)
- added REF**: OSMU_logo, bitaxe:OSMU_logo, F.Cu at (54.9, 132.8)
