File: bm1366-1.kicad_sch (KiCad schematic)
At the start: 54 parts, among them U1 25MHz, U10 AP7331, U11 AP7331, U12 BM1368_mode1, U28 BM1368_mode1

Commit message: init push for GammaHex
Parts:
- removed U12, U28: BM1368_mode1, bitaxe:BM1368, symbol bitaxe:BM1368_mode1
- added U12, U22: BM1370_mode1, bitaxe:BM1370, symbol bitaxe:BM1370_mode1
Connections:
- net 0V8: now also U12.14 (VDDIO_08_0), U12.17 (VDDIO_08_1), U22.14 (VDDIO_08_0), U22.17 (VDDIO_08_1)
- net 1V8: now also U12.15 (VDDIO_12_0), U12.16 (VDDIO_12_1), U22.15 (VDDIO_12_0), U22.16 (VDDIO_12_1)
- net BI1: now also U12.9 (BI)
- net BO: now also U22.22 (BO)
- net CI: now also U12.6 (CI)
- net CLKI1: now also U12.8 (CLKI)
- net CO: now also U22.25 (CO)
- net GND1: now also U12.13 (PLL_VSS), U12.18 (VSS), U12.27 (VSS), U12.32 (VSS), U12.4 (VSS), U22.13 (PLL_VSS), U22.18 (VSS), U22.27 (VSS), U22.32 (VSS), U22.4 (VSS)
- net NRSTI: now also U12.5 (NRSTI)
- net NRSTO: now also U22.26 (NRSTO)
- net RI: now also U22.24 (RI)
- net RO: now also U12.7 (RO)
- net TEMP_N1: now also U12.21 (TEMP_N)
- net TEMP_N2: now also U22.21 (TEMP_N)
- net TEMP_P1: now also U12.20 (TEMP_P)
- net TEMP_P2: now also U22.20 (TEMP_P)
- net VDD1: now also U12.31 (VDD), U22.31 (VDD)
- net at C2.2, C3.1: now also U12.3 (VDD1_0)
- net at C12.2, C15.1, C6.2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: now also U12.30 (VDD3_1), U22.1 (VDD3_0)
- net at TP13.1: now also U22.10 (ROSC_SEL)
- net at R79.2: now also U22.11 (LITE_PAD)
- net at TP13.1: now also U22.12 (INV_CLKO)
- net at C15.2, C17.1, C3.2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: now also U12.29 (VDD2_1), U22.2 (VDD2_0)
- net at TP13.1: now also U22.23 (CLKO)
- net at C17.2, C18.1: now also U22.28 (VDD1_1)
- net at C15.2, C17.1: now also U22.29 (VDD2_1)
- net at C17.2, C18.1, C2.2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: now also U12.28 (VDD1_1), U22.3 (VDD1_0)
- net at C12.2, C15.1: now also U22.30 (VDD3_1)
- net at R6.2: now also U12.26 (NRSTO), U22.5 (NRSTI)
- net at C6.2, C8.1: now also U12.1 (VDD3_0)
- net at C3.2, C6.1: now also U12.2 (VDD2_0)
- net at TP13.1: now also U12.10 (ROSC_SEL)
- net at R78.2: now also U12.11 (LITE_PAD)
- net at TP13.1: now also U12.12 (INV_CLKO)
- new net: U12.25 (CO), U22.6 (CI)
- new net: U12.24 (RI), U22.7 (RO)
- new net: U12.23 (CLKO), U22.8 (CLKI)
- new net: U12.22 (BO), U22.9 (BI)
